File: bep.sch (KiCad schematic (older format))
At the start: 0 parts

Commit message: add local symbol library, begin schematic
Parts:
- added C?: 4.7u, symbol Device:C
- added D? (x8): D, symbol Device:D
- added D?: LED, symbol Device:LED
- added J?: Conn_01x24, symbol Connector_Generic:Conn_01x24
- added JP? (x5): Jumper, symbol Device:Jumper
- added Q? (x2): SMBTA42, Package_TO_SOT_SMD:SOT-23, symbol Device:Q_NPN_BEC
- added Q?: BCP51, Package_TO_SOT_SMD:SOT-223, symbol Transistor_BJT:BCP51
- added R?: 4.7k, symbol Device:R
- added R? (x5): 10k, symbol Device:R
- added R?: 350, symbol Device:R
- added R?: 1k, symbol Device:R
- added U?: LTC2054, Package_TO_SOT_SMD:TSOT-23-5_HandSoldering, symbol bep:LTC2054
Connections:
- net labels added: +12V, +5V, 12V, ABS_LAMP, BCD_NEUTRAL, CHARGING_LAMP, CHOKE_LAMP, COMBINED_WARNING_LAMP, GEAR_BCD_A, GEAR_BCD_B, GEAR_BCD_C, GND, HIGH_BEAM, LIGHT_CHECK_LAMP, OIL_LAMP, RPM_COIL, RPM_SIGNAL, SPEED_SENSOR, SPEED_SIGNAL, START_BUTTON, TEMP_LAMP, TURN_BOTH_OUT, TURN_L, TURN_L_OUT, TURN_R, TURN_R_OUT
- wire segments 0 -> 96
- no-connect marks 0 -> 1
Other:
- note added: "12V Battery"
- note added: "12V Ignition"
- note added: "12V for start button"
- note added: "12V/350mA to start button"
- note added: "5V for OpAmp"
- note added: "ABS lamp"
- note added: "Charging control lamp"
- note added: "Choke lamp"
- note added: "Combine several warning lamps into one"
- note added: "Combine turn signals if only one indicator for both L and R is available"
- note added: "Fuel reserve lamp"
- note added: "GND"
- note added: "Gear Signal A"
- note added: "Gear Signal B"
- note added: "Gear Signal C"
- note added: "High beam"
- note added: "INPUT"
- note added: "INSERT 5V LDO here"
- note added: "Instrument illumination (12V Ignition)"
- note added: "K100 Lunchbox Adapter"
- note added: "Light check lamp"
- note added: "NC"
- note added: "OUTPUT"
- note added: "Oil pressure lamp"
- note added: "RPM ignition coil"
- note added: "Speed sensor GND"
- note added: "Speed sensor signal"
- note added: "Speed signal conversion to rect wave"
- note added: "Speed signal to turn signal relais"
- note added: "Temperature lamp"
- note added: "Turn signal left"
- note added: "Turn signal right"
