File: bep.kicad_pcb (KiCad board)
At the start: 2 copper layers, 76 parts, among them J1 Conn_01x12, J2 Conn_01x24, J3 Conn_01x12, Q1 SMBTA42, Q10 SMBTA42, Q11 SMBTA42, Q2 SMBTA42, Q3 SMBTA42, Q4 SMBTA42, Q5 SMBTA42, Q6 SMBTA42, Q7 BCP51, Q8 SMBTA42, Q9 SMBTA42, U1 HCF4028B, U2 LM1117-5.0, U3 LM2904

Commit message: begin pcb
Parts:
- removed the C5 at (145.7, 161.0)
- removed the D15 at (74.6, 162.4)
- removed the J2 at (63.5, 59.2)
- removed the R13 at (185.1, 103.4)
- removed the R17 at (111.4, 146.6)
- removed the R25 at (143.3, 120.6)
- removed the R32 at (82.0, 55.9)
- added C4: 100n, Capacitor_THT:C_Rect_L18.0mm_W8.0mm_P15.00mm_FKS3_FKP3, F.Cu at (59.7, 33.0)
- added D1: D, Diode_SMD:D_0603_1608Metric_Pad1.05x0.95mm_HandSolder, F.Cu at (76.2, 67.7)
- added J3: Conn_01x03, Connector_PinHeader_2.54mm:PinHeader_1x03_P2.54mm_Vertical, F.Cu at (103.0, 29.8)
- added J4: Conn_01x03, Connector_PinHeader_2.54mm:PinHeader_1x04_P2.54mm_Vertical, F.Cu at (113.0, 116.8)
- added J5: Conn_01x03, Connector_PinHeader_2.54mm:PinHeader_1x04_P2.54mm_Vertical, F.Cu at (231.1, 33.0)
- added J6: Conn_01x06, Connector_PinHeader_2.54mm:PinHeader_1x06_P2.54mm_Vertical, F.Cu at (84.4, 29.8)
- added J7: Conn_01x06, Connector_PinHeader_2.54mm:PinHeader_1x06_P2.54mm_Vertical, F.Cu at (225.4, 132.1)
- added J8: Conn_01x03, Connector_PinHeader_2.54mm:PinHeader_1x03_P2.54mm_Vertical, F.Cu at (224.2, 95.9)
- added JP3: Jumper_3_Bridged12, Connector_PinHeader_2.54mm:PinHeader_1x03_P2.54mm_Vertical, F.Cu at (219.7, 35.6)
- added Q12: SMBTA42, Package_TO_SOT_SMD:SOT-23, F.Cu at (212.4, 30.5)
- added R15: 10k, Resistor_SMD:R_0805_2012Metric_Pad1.15x1.40mm_HandSolder, F.Cu at (47.9, 144.1)
- added R21: 4.7k, Resistor_SMD:R_0805_2012Metric_Pad1.15x1.40mm_HandSolder, F.Cu at (207.0, 41.9)
- added R29: 10k, Resistor_SMD:R_0805_2012Metric_Pad1.15x1.40mm_HandSolder, F.Cu at (61.2, 101.6)
- added R31: 10k, Resistor_SMD:R_0805_2012Metric_Pad1.15x1.40mm_HandSolder, F.Cu at (219.7, 31.5)
- added R33: 10k, Resistor_SMD:R_0805_2012Metric_Pad1.15x1.40mm_HandSolder, F.Cu at (224.8, 31.5)
- C1: value 100n -> 10u; footprint Capacitor_SMD:C_1206_3216Metric_Pad1.42x1.75mm_HandSolder -> Capacitor_SMD:CP_Elec_4x5.8
- C3: value 10u -> 100n; footprint Capacitor_SMD:CP_Elec_4x5.8 -> Capacitor_SMD:C_1206_3216Metric_Pad1.42x1.75mm_HandSolder
- moved R1 175.1 mm to (41.5, 136.5)
- moved R14 169.4 mm to (67.6, 136.5)
- moved Q3 165.3 mm to (51.8, 147.7), turned to 270 degrees
- moved D14 161.5 mm to (219.7, 96.8), turned to 90 degrees
- moved JP2 157.1 mm to (224.8, 39.4), turned to 270 degrees
- moved R2 154.8 mm to (41.5, 134.0)
- moved Q1 153.1 mm to (48.6, 129.2), turned to 90 degrees
- moved R3 152.2 mm to (41.5, 139.1)
- moved Q4 149.7 mm to (56.2, 129.2), turned to 90 degrees
- moved R13 149.3 mm to (60.3, 139.7), turned to 90 degrees
- moved Q8 147.9 mm to (52.4, 129.2), turned to 90 degrees
- moved R4 146.1 mm to (48.3, 132.7), turned to 180 degrees
- moved R11 144.6 mm to (56.3, 132.7), turned to 180 degrees
- moved U3 138.0 mm to (213.4, 41.9)
- moved U1 133.5 mm to (52.7, 138.4), turned to 270 degrees
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- renumbered C4 to C2, C6 to C5, C2 to C6, D8 to D10, D9 to D11, D10 to D12, D16 to D13, D11 to D14, D12 to D15, D13 to D16, D1 to D2, D2 to D3, D3 to D4, D4 to D5, D5 to D6, D6 to D7, D14 to D8, D7 to D9, J3 to J2, Q11 to Q10, Q9 to Q11, Q7 to Q5, Q8 to Q6, Q5 to Q7, Q6 to Q8, Q10 to Q9, R21 to R13, R22 to R14, R24 to R16, R14 to R17, R20 to R18, R26 to R19, R27 to R20, R28 to R22, R29 to R23, R18 to R24, R30 to R25, R19 to R26, R31 to R27, R23 to R28, R15 to R30, R16 to R32, R33 to R34
Connections:
- net /BCD_NEUTRAL renamed BCD_NEUTRAL
- net /CHARGING_LAMP renamed CHARGE_LAMP
- net /CHOKE_LAMP renamed CHOKE_LAMP
- net /COMBINED_WARNING_LAMP renamed WRNG_LAMP
- net /GEAR_BCD_A renamed GEAR_BCD_A
- net /GEAR_BCD_B renamed GEAR_BCD_B
- net /GEAR_BCD_C renamed GEAR_BCD_C
- net /LIGHT_CHECK_LAMP renamed LIGHT_LAMP
- net /OIL_LAMP renamed OIL_LAMP
- net /SPEED_SIGNAL renamed SPD_12V
- net /START_BUTTON renamed START_BUTTON
- net /TEMP_LAMP renamed TEMP_LAMP
- net /TURN_BOTH_OUT renamed Net-(D14-Pad1)
- net /TURN_L renamed TURN_L
- net /TURN_R renamed TURN_R
- C1 pad 1: +12V -> Net-(C1-Pad1)
- C3 pad 1: Net-(C3-Pad1) -> +12V
- D2 pad 1: Net-(C3-Pad1) -> Net-(C1-Pad1)
- J1 pad 8: /ABS_LAMP -> Net-(J1-Pad8)
- J2 pad 10: /SPEED_SENSOR -> SPEED_SENSOR
- J2 pad 3: /HIGH_BEAM -> Net-(J2-Pad3)
- J2 pad 4: /RPM_COIL -> RPM_COIL
- JP2 pad 2: /RPM_SIGNAL -> RPM
- Q1 pad 3: /GEAR5 -> GEAR_5
- Q2 pad 3: /GEAR4 -> GEAR_4
- Q3 pad 3: /GEAR3 -> GEAR_3
- Q4 pad 3: /GEAR2 -> GEAR_2
- Q7 pad 3: /GEAR1 -> GEAR_1
- Q8 pad 3: /GEAR_NEUTRAL -> GEAR_N
- U2 pad 3: Net-(C3-Pad1) -> Net-(C1-Pad1)

Commit message: finished pcb, review candidate
Parts:
- removed J2: Conn_01x12, Connector_PinHeader_2.54mm:PinHeader_1x12_P2.54mm_Vertical
- added REF**: MountingHole_3.2mm_M3_DIN965_Pad, MountingHole:MountingHole_3.2mm_M3_DIN965_Pad, F.Cu at (165.4, 111.5)
- added REF**: MountingHole_3.2mm_M3_DIN965_Pad, MountingHole:MountingHole_3.2mm_M3_DIN965_Pad, F.Cu at (177.7, 53.1)
- added REF**: MountingHole_3.2mm_M3_DIN965_Pad, MountingHole:MountingHole_3.2mm_M3_DIN965_Pad, F.Cu at (131.1, 76.3)
- added REF**: MountingHole_3.2mm_M3_DIN965_Pad, MountingHole:MountingHole_3.2mm_M3_DIN965_Pad, F.Cu at (131.1, 95.4)
- added REF**: KiCad-Logo_5mm_SilkScreen, Symbol:KiCad-Logo_5mm_SilkScreen, F.Cu at (123.3, 127.0)
- added REF**: MountingHole_3.2mm_M3_DIN965_Pad, MountingHole:MountingHole_3.2mm_M3_DIN965_Pad, F.Cu at (118.7, 53.1)
- added REF**: MountingHole_3.2mm_M3_DIN965_Pad, MountingHole:MountingHole_3.2mm_M3_DIN965_Pad, F.Cu at (176.3, 87.9)
- added REF**: MountingHole_3.2mm_M3_DIN965_Pad, MountingHole:MountingHole_3.2mm_M3_DIN965_Pad, F.Cu at (118.4, 134.0)
- C4: footprint Capacitor_THT:C_Rect_L18.0mm_W8.0mm_P15.00mm_FKS3_FKP3 -> Capacitor_SMD:C_1206_3216Metric_Pad1.42x1.75mm_HandSolder
- J1: value Conn_01x12 -> Conn_01x24; footprint Connector_PinHeader_2.54mm:PinHeader_1x12_P2.54mm_Vertical -> bep:DIP-24_866
- R30: value 47 2W -> 100 1.6W; footprint Resistor_THT:R_Axial_DIN0614_L14.3mm_D5.7mm_P25.40mm_Horizontal -> Resistor_SMD:R_1206_3216Metric_Pad1.42x1.75mm_HandSolder
- R31: value 10k -> 100 1.6W; footprint Resistor_SMD:R_0805_2012Metric_Pad1.15x1.40mm_HandSolder -> Resistor_SMD:R_1206_3216Metric_Pad1.42x1.75mm_HandSolder
- R32: value 47 2W -> 10k; footprint Resistor_THT:R_Axial_DIN0614_L14.3mm_D5.7mm_P25.40mm_Horizontal -> Resistor_SMD:R_0805_2012Metric_Pad1.15x1.40mm_HandSolder
- moved R30 157.3 mm to (131.7, 54.9), turned to 90 degrees
- moved Q3 138.1 mm to (167.4, 72.3), turned to 0 degrees
- moved Q7 137.4 mm to (167.4, 79.9), turned to 0 degrees
- moved Q2 137.0 mm to (167.4, 68.5), turned to 0 degrees
- moved Q1 135.2 mm to (167.4, 64.6), turned to 0 degrees
- moved R7 134.5 mm to (163.1, 68.5), turned to 0 degrees
- moved R4 133.9 mm to (163.1, 63.9), turned to 0 degrees
- moved R6 132.6 mm to (163.1, 66.2), turned to 0 degrees
- moved R15 130.8 mm to (163.1, 82.2), turned to 0 degrees
- moved R2 128.4 mm to (158.8, 81.7), turned to 90 degrees
- moved R1 127.2 mm to (156.2, 81.7), turned to 90 degrees
- moved R3 126.0 mm to (153.7, 81.7), turned to 90 degrees
- moved D16 124.6 mm to (148.0, 52.8), turned to 270 degrees
- moved Q8 123.7 mm to (167.4, 83.7), turned to 0 degrees
- moved U1 123.5 mm to (158.1, 74.0)
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Connections:
- J4 pad 4: Net-(J2-Pad3) -> Net-(J1-Pad15)
- R30 pad 1: Net-(R30-Pad1) -> +12V
- R31 pad 1: SPD_12V -> +12V
- R31 pad 2: +12V -> Net-(D16-Pad2)
- R32 pad 1: +12V -> SPD_12V
- R32 pad 2: Net-(R30-Pad1) -> +12V
Routing:
- net SPD_12V: track 0.00 -> 114.7 mm, vias 0 -> 1
- net SPEED_SENSOR: track 0.00 -> 97.8 mm, vias 0 -> 1
- net GND: track 0.00 -> 87.1 mm, vias 0 -> 15
- net CHARGE_LAMP: track 0.00 -> 85.3 mm
- net TEMP_LAMP: track 0.00 -> 76.4 mm
- net CHOKE_LAMP: track 0.00 -> 76.3 mm
- net OIL_LAMP: track 0.00 -> 75.8 mm
- net +12V: track 0.00 -> 75.0 mm, vias 0 -> 12
- net Net-(J1-Pad8): track 0.00 -> 74.1 mm
- net LIGHT_LAMP: track 0.00 -> 73.0 mm, vias 0 -> 2
- net Net-(J1-Pad1): track 0.00 -> 71.6 mm
- net Net-(J1-Pad7): track 0.00 -> 64.8 mm
- net START_BUTTON: track 0.00 -> 57.9 mm, vias 0 -> 1
- net TURN_L: track 0.00 -> 51.1 mm
- net GEAR_BCD_C: track 0.00 -> 50.4 mm, vias 0 -> 1
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- added copper zone on F.Cu, net +12V
- added copper zone on B.Cu, net GND
Other:
- board outline added: 67.6 x 89.2 mm
- board text added: "1"
- board text added: "12V"
- board text added: "2"
- board text added: "3"
- board text added: "4"
- board text added: "5"
- board text added: "ABS"
- board text added: "Adapter"
- board text added: "BAT"
- board text added: "Beam"
- board text added: "CHK"
- board text added: "GND"
- board text added: "Gauges"
- board text added: "Gears"
- board text added: "HI"
- board text added: "L"
- board text added: "LGHT"
- board text added: "Lamps"
- board text added: "Lunchbox"
- board text added: "N"
- board text added: "OIL"
- board text added: "Power"
- board text added: "R"
- board text added: "R+L"
- board text added: "RPM"
- board text added: "RSV"
- board text added: "SPD"
- board text added: "TMP"
- board text added: "Turn Signals"
- board text added: "VCC"
- board text added: "WRN"
- board text added: "Warning Lamps"
- board text added: "const"
- board text added: "ign"
- board text added: "v1.0"
