File: lunchbox-adapter.sch (KiCad schematic (older format))
At the start: 83 parts, among them J1 Conn_01x24, J3 Conn_01x03, J4 Conn_01x03, J5 Conn_01x03, J6 Conn_01x06, J7 Conn_01x06, J8 Conn_01x03, Q1 SMBTA42, Q10 SMBTA42, Q11 SMBTA42, Q12 SMBTA42, Q2 SMBTA42, Q3 SMBTA42, Q4 SMBTA42, Q5 BCP51, Q6 SMBTA42, Q7 SMBTA42, Q8 SMBTA42, Q9 SMBTA42, U1 HCF4028B, U2 LM1117-5.0, U3 LM2904

Commit message: finished pcb design
Changed lines of the file:
@@
 EESchema Schematic File Version 4
-LIBS:bep-cache
 EELAYER 29 0
 EELAYER END
@@
 U 1 1 5D19D05C
 P 9950 5200
-F 0 "R30" V 9743 5200 50  0000 C CNN
-F 1 "100 1.6W" V 9900 5400 50  0000 C CNN
+F 0 "R30" V 9850 5150 50  0000 C CNN
+F 1 "100 1.6W" V 9850 5450 50  0000 C CNN
 F 2 "Resistor_SMD:R_1206_3216Metric_Pad1.42x1.75mm_HandSolder" V 9880 5200 50  0001 C CNN
 F 3 "~" H 9950 5200 50  0001 C CNN
@@
 U 1 1 5D1A0765
 P 9950 5400
-F 0 "R31" V 10050 5400 50  0000 C CNN
-F 1 "100 1.6W" V 10000 5600 50  0000 C CNN
+F 0 "R31" V 10050 5350 50  0000 C CNN
+F 1 "100 1.6W" V 10050 5650 50  0000 C CNN
 F 2 "Resistor_SMD:R_1206_3216Metric_Pad1.42x1.75mm_HandSolder" V 9880 5400 50  0001 C CNN
 F 3 "~" H 9950 5400 50  0001 C CNN

Commit message: change power resitor footprints, cleanup
Parts:
- R30, R31: footprint Resistor_SMD:R_1206_3216Metric_Pad1.42x1.75mm_HandSolder -> bep:5020_resistor_thermal_pads
Changed lines of the file:
@@
 EESchema Schematic File Version 4
+LIBS:lunchbox-adapter-cache
 EELAYER 29 0
 EELAYER END
@@
 F 0 "R30" V 9850 5150 50  0000 C CNN
 F 1 "100 1.6W" V 9850 5450 50  0000 C CNN
-F 2 "Resistor_SMD:R_1206_3216Metric_Pad1.42x1.75mm_HandSolder" V 9880 5200 50  0001 C CNN
+F 2 "bep:5020_resistor_thermal_pads" V 9880 5200 50  0001 C CNN
 F 3 "~" H 9950 5200 50  0001 C CNN
 	1    9950 5200
@@
 F 0 "R31" V 10050 5350 50  0000 C CNN
 F 1 "100 1.6W" V 10050 5650 50  0000 C CNN
-F 2 "Resistor_SMD:R_1206_3216Metric_Pad1.42x1.75mm_HandSolder" V 9880 5400 50  0001 C CNN
+F 2 "bep:5020_resistor_thermal_pads" V 9880 5400 50  0001 C CNN
 F 3 "~" H 9950 5400 50  0001 C CNN
 	1    9950 5400
